File: boards/esc/motor_driver_phase_A.kicad_sch (KiCad schematic)
At the start: 13 parts, among them Q8 BSC340N08NS3G, U2 MIC4605-2YM-TR

Commit message: started simplified esc
Connections:
- net PHASE_A: now also C7.2, U2.4 (HS)
Changed lines of the file:
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@@
   (junction (at 152.4 101.6) (diameter 0) (color 0 0 0 0)
+  )
+  (junction (at 107.95 76.2) (diameter 0) (color 0 0 0 0)
   )
   (junction (at 160.02 101.6) (diameter 0) (color 0 0 0 0)
@@
   )
   (wire (pts (xy 128.27 57.15) (xy 128.27 69.85))
+    (stroke (width 0) (type default))
+  )
+  (wire (pts (xy 107.95 76.2) (xy 121.92 76.2))
     (stroke (width 0) (type default))
   )
@@
   )
   (wire (pts (xy 134.62 63.5) (xy 134.62 64.77))
+    (stroke (width 0) (type default))
+  )
+  (wire (pts (xy 121.92 81.28) (xy 128.27 81.28))
     (stroke (width 0) (type default))
   )
@@
     (stroke (width 0) (type default))
   )
+  (wire (pts (xy 121.92 76.2) (xy 121.92 81.28))
+    (stroke (width 0) (type default))
+  )
